Commit message: WIP

File: multi_turtlebot_gazebo/world/models/robot/config/turtlebot_properties.urdf.xacro (robot description, xacro)
@@ -19,7 +19,9 @@
      (currently in development and awaiting feedback)
    -->
-  <xacro:property name="cam_px" value="-0.035" />
+  <!-- <xacro:property name="cam_px" value="-0.035" /> -->
+  <xacro:property name="cam_px" value="0.05" />
 <!--	<xacro:property name="cam_py" value="-0.0125" /> Y varies for different configurations. get sets in sensors_urdf -->
-  <xacro:property name="cam_pz" value="0.390" />
+  <!-- <xacro:property name="cam_pz" value="0.390" /> -->
+  <xacro:property name="cam_pz" value="0.0" />
 	<xacro:property name="cam_or" value="0" />
 	<xacro:property name="cam_op" value="0" />

File: multi_turtlebot_gazebo/world/models/robot/labs_turtlebot2.urdf.xacro (robot description, xacro)
@@ -12,4 +12,4 @@
   <kobuki/>
   <stack_hexagons parent="base_link"/>
-  <sensor_kinect  parent="base_link"/>
+  <sensor_kinect  parent="merge_laser_link"/>
 </robot>

Commit message: edit urdf and launch

File: multi_turtlebot_gazebo/world/models/robot/config/turtlebot_properties.urdf.xacro (robot description, xacro)
@@ -19,4 +19,5 @@
      (currently in development and awaiting feedback)
    -->
+   <xacro:include filename="$(find turtlebot_description)/urdf/common_properties.urdf.xacro"/>
   <!-- <xacro:property name="cam_px" value="-0.035" /> -->
   <xacro:property name="cam_px" value="0.05" />
@@ -28,8 +29,8 @@
 	<xacro:property name="cam_oy" value="0" />
   <xacro:property name="urg_px" value="0.05" />
-<!--	<xacro:property name="urg_py" value="-0.0125" /> Y varies for different configurations. get sets in sensors_urdf -->
+	<xacro:property name="urg_py" value="0.0" />
   <xacro:property name="urg_pz" value="0.0" />
-	<xacro:property name="urg_or" value="0" />
-	<xacro:property name="urg_op" value="0" />
-	<xacro:property name="urg_oy" value="3.1416" />
+	<xacro:property name="urg_or" value="0.0" />
+	<xacro:property name="urg_op" value="0.0" />
+	<xacro:property name="urg_oy" value="${M_PI}" />
 </robot>

File: multi_turtlebot_gazebo/world/models/robot/config/urg.urdf.xacro (robot description, xacro)
@@ -1,5 +1,4 @@
 <?xml version="1.0"?>
 <robot name="sensor_urg" xmlns:xacro="http://ros.org/wiki/xacro">
-  <xacro:include filename="$(find turtlebot_description)/urdf/turtlebot_gazebo.urdf.xacro"/>
   <xacro:include filename="$(find multi_turtlebot_gazebo)/world/models/robot/config/turtlebot_properties.urdf.xacro"/>
   <xacro:macro name="sensor_urg" params="parent">

File: multi_turtlebot_gazebo/world/models/robot/labs_turtlebot2.urdf.xacro (robot description, xacro)
@@ -9,5 +9,5 @@
   <xacro:include filename="$(find kobuki_description)/urdf/kobuki.urdf.xacro" />
   <xacro:include filename="$(find multi_turtlebot_gazebo)/world/models/robot/config/hexagons.urdf.xacro"/>
-  <xacro:include filename="$(find turtlebot_description)/urdf/sensors/kinect.urdf.xacro"/>
+  <xacro:include filename="$(find multi_turtlebot_gazebo)/world/models/robot/config/kinect.urdf.xacro"/>
   <kobuki/>
   <stack_hexagons parent="base_link"/>

File: multi_turtlebot_gazebo/world/models/robot/labs_turtlebot2_urg.urdf.xacro (robot description, xacro)
@@ -9,5 +9,5 @@
   <xacro:include filename="$(find multi_turtlebot_gazebo)/world/models/robot/config/kobuki_urg.urdf.xacro" />
   <xacro:include filename="$(find multi_turtlebot_gazebo)/world/models/robot/config/hexagons.urdf.xacro"/>
-  <xacro:include filename="$(find turtlebot_description)/urdf/sensors/kinect.urdf.xacro"/>
+  <xacro:include filename="$(find multi_turtlebot_gazebo)/world/models/robot/config/kinect.urdf.xacro"/>
   <xacro:include filename="$(find multi_turtlebot_gazebo)/world/models/robot/config/urg.urdf.xacro"/>
   <kobuki/>

Commit message: minor fix

File: multi_turtlebot_gazebo/world/models/robot/config/turtlebot_properties.urdf.xacro (robot description, xacro)
@@ -28,5 +28,5 @@
 	<xacro:property name="cam_op" value="0" />
 	<xacro:property name="cam_oy" value="0" />
-  <xacro:property name="urg_px" value="0.05" />
+  <xacro:property name="urg_px" value="-0.05" />
 	<xacro:property name="urg_py" value="0.0" />
   <xacro:property name="urg_pz" value="0.0" />

File: multi_turtlebot_gazebo/world/models/robot/config/urg.urdf.xacro (robot description, xacro)
@@ -4,5 +4,5 @@
   <xacro:macro name="sensor_urg" params="parent">
     <joint name="urg_joint" type="fixed">
-      <origin xyz="${urg_px} ${urg_py} ${urg_pz}" rpy="${urg_ox} ${urg_oy} ${urg_oz}" />
+      <origin xyz="${urg_px} ${urg_py} ${urg_pz}" rpy="${urg_or} ${urg_op} ${urg_oy}" />
       <parent link="${parent}" />
       <child link="urg_frame" />

Commit message: minor fix

File: multi_turtlebot_gazebo/world/models/robot/config/turtlebot_properties.urdf.xacro (robot description, xacro)
@@ -21,5 +21,5 @@
    <xacro:include filename="$(find turtlebot_description)/urdf/common_properties.urdf.xacro"/>
   <!-- <xacro:property name="cam_px" value="-0.035" /> -->
-  <xacro:property name="cam_px" value="0.05" />
+  <xacro:property name="cam_px" value="0.07" />
 <!--	<xacro:property name="cam_py" value="-0.0125" /> Y varies for different configurations. get sets in sensors_urdf -->
   <!-- <xacro:property name="cam_pz" value="0.390" /> -->
@@ -28,5 +28,5 @@
 	<xacro:property name="cam_op" value="0" />
 	<xacro:property name="cam_oy" value="0" />
-  <xacro:property name="urg_px" value="-0.05" />
+  <xacro:property name="urg_px" value="-0.06" />
 	<xacro:property name="urg_py" value="0.0" />
   <xacro:property name="urg_pz" value="0.0" />

Commit message: fix urdf param

File: multi_turtlebot_gazebo/world/models/robot/config/turtlebot_properties.urdf.xacro (robot description, xacro)
@@ -22,4 +22,5 @@
   <!-- <xacro:property name="cam_px" value="-0.035" /> -->
   <xacro:property name="cam_px" value="0.07" />
+  <!-- <xacro:property name="cam_px" value="0.00" /> -->
 <!--	<xacro:property name="cam_py" value="-0.0125" /> Y varies for different configurations. get sets in sensors_urdf -->
   <!-- <xacro:property name="cam_pz" value="0.390" /> -->

File: multi_turtlebot_gazebo/world/models/robot/labs_turtlebot2.urdf.xacro (robot description, xacro)
@@ -9,5 +9,6 @@
   <xacro:include filename="$(find kobuki_description)/urdf/kobuki.urdf.xacro" />
   <xacro:include filename="$(find multi_turtlebot_gazebo)/world/models/robot/config/hexagons.urdf.xacro"/>
-  <xacro:include filename="$(find multi_turtlebot_gazebo)/world/models/robot/config/kinect.urdf.xacro"/>
+  <!-- <xacro:include filename="$(find multi_turtlebot_gazebo)/world/models/robot/config/kinect.urdf.xacro"/> -->
+  <xacro:include filename="$(find turtlebot_description)/urdf/sensors/kinect.urdf.xacro"/>
   <kobuki/>
   <stack_hexagons parent="base_link"/>
