Commit message: change parameter

File: multi_turtlebot_gazebo/world/models/robot/config/turtlebot_properties_urg.urdf.xacro (robot description, xacro)
@@ -20,12 +20,18 @@
    -->
    <xacro:include filename="$(find turtlebot_description)/urdf/common_properties.urdf.xacro"/>
-  <xacro:property name="cam_px" value="-0.035" />
-  <!-- <xacro:property name="cam_px" value="0" /> -->
+  <!-- <xacro:property name="cam_px" value="-0.035" /> -->
+  <xacro:property name="cam_px" value="0.07" />
   <!-- <xacro:property name="cam_px" value="0.00" /> -->
 <!--	<xacro:property name="cam_py" value="-0.0125" /> Y varies for different configurations. get sets in sensors_urdf -->
-  <xacro:property name="cam_pz" value="0.390" />
-  <xacro:property name="cam_pz" value="0" />
+  <!-- <xacro:property name="cam_pz" value="0.390" /> -->
+  <xacro:property name="cam_pz" value="0.0" />
 	<xacro:property name="cam_or" value="0" />
 	<xacro:property name="cam_op" value="0" />
 	<xacro:property name="cam_oy" value="0" />
+  <xacro:property name="urg_px" value="-0.06" />
+	<xacro:property name="urg_py" value="0.0" />
+  <xacro:property name="urg_pz" value="0.0" />
+	<xacro:property name="urg_or" value="0.0" />
+	<xacro:property name="urg_op" value="0.0" />
+	<xacro:property name="urg_oy" value="${M_PI}" />
 </robot>

File: multi_turtlebot_gazebo/world/models/robot/labs_turtlebot2_urg.urdf.xacro (robot description, xacro)
@@ -6,8 +6,8 @@
 -->
 <robot name="turtlebot" xmlns:xacro="http://ros.org/wiki/xacro">
-  <xacro:include filename="$(find multi_turtlebot_gazebo)/world/models/robot/config/turtlebot_common_library.urdf.xacro" />
+  <xacro:include filename="$(find multi_turtlebot_gazebo)/world/models/robot/config/turtlebot_common_library_urg.urdf.xacro" />
   <xacro:include filename="$(find multi_turtlebot_gazebo)/world/models/robot/config/kobuki_urg.urdf.xacro" />
   <xacro:include filename="$(find multi_turtlebot_gazebo)/world/models/robot/config/hexagons.urdf.xacro"/>
-  <xacro:include filename="$(find multi_turtlebot_gazebo)/world/models/robot/config/kinect.urdf.xacro"/>
+  <xacro:include filename="$(find multi_turtlebot_gazebo)/world/models/robot/config/kinect_urg.urdf.xacro"/>
   <xacro:include filename="$(find multi_turtlebot_gazebo)/world/models/robot/config/urg.urdf.xacro"/>
   <kobuki/>
