Commit message: fix urdf

File: lab_turtlebot_description/urdf/config/turtlebot_properties.urdf.xacro (robot description, xacro)
@@ -25,5 +25,5 @@
 <!--	<xacro:property name="cam_py" value="-0.0125" /> Y varies for different configurations. get sets in sensors_urdf -->
   <xacro:property name="cam_pz" value="0.390" />
-  <xacro:property name="cam_pz" value="0" />
+  <!-- <xacro:property name="cam_pz" value="0" /> -->
 	<xacro:property name="cam_or" value="0" />
 	<xacro:property name="cam_op" value="0" />
