Commit message: add steleo

File: lab_turtlebot_description/urdf/config/hexagons.urdf.xacro (robot description, xacro)
@@ -4,5 +4,5 @@
  -->
 <robot name="stack_hexagons" xmlns:xacro="http://ros.org/wiki/xacro">
-  <xacro:include filename="$(find turtlebot_description)/urdf/common_properties.urdf.xacro"/>
+  <xacro:include filename="$(find lab_turtlebot_description)/urdf/config/common_properties.urdf.xacro"/>
   <!-- Xacro properties -->
   <xacro:property name="M_SCALE" value="0.001"/>

File: lab_turtlebot_description/urdf/config/steleo.urdf.xacro (robot description, xacro)
@@ -1,5 +1,5 @@
 <?xml version="1.0"?>
 <robot name="sensor_kinect" xmlns:xacro="http://ros.org/wiki/xacro">
-  <xacro:include filename="$(find lab_turtlebot_description)/urdf/config/turtlebot_gazebo_kinect.urdf.xacro"/>
+  <xacro:include filename="$(find lab_turtlebot_description)/urdf/config/turtlebot_gazebo_steleo.urdf.xacro"/>
   <xacro:include filename="$(find lab_turtlebot_description)/urdf/config/turtlebot_properties.urdf.xacro"/>
   <xacro:property name="kinect_cam_py" value="-0.0125"/>
@@ -21,7 +21,7 @@
       <origin xyz="-0.031 ${-kinect_cam_py} -0.016" rpy="0 0 0"/>
       <parent link="camera_rgb_frame"/>
-      <child link="camera_link"/>
+      <child link="left_camera_frame"/>
     </joint>
-      <link name="camera_link">
+      <link name="left_camera_frame">
       <visual>
        <origin xyz="0 0 0" rpy="0 0 ${M_PI/2}"/>

File: lab_turtlebot_description/urdf/config/turtlebot_common_library.urdf.xacro (robot description, xacro)
@@ -5,5 +5,5 @@
 <robot xmlns:xacro="http://ros.org/wiki/xacro">
   <!-- General -->
-  <xacro:include filename="$(find turtlebot_description)/urdf/common_properties.urdf.xacro"/>
+  <xacro:include filename="$(find lab_turtlebot_description)/urdf/config/common_properties.urdf.xacro"/>
   <xacro:include filename="$(find lab_turtlebot_description)/urdf/config/turtlebot_properties.urdf.xacro"/>
 </robot>
