Commit message: lab_turtlebot_description

File: lab_turtlebot_description/urdf/config/kinect/kinect.urdf.xacro (robot description, xacro)
@@ -1,9 +1,9 @@
 <?xml version="1.0"?>
-<robot name="sensor_steleo" xmlns:xacro="http://ros.org/wiki/xacro">
-  <xacro:include filename="$(find lab_turtlebot_description)/urdf/config/turtlebot_gazebo_steleo.urdf.xacro"/>
-  <xacro:include filename="$(find lab_turtlebot_description)/urdf/config/turtlebot_properties.urdf.xacro"/>
+<robot name="sensor_kinect" xmlns:xacro="http://ros.org/wiki/xacro">
+  <xacro:include filename="$(find lab_turtlebot_description)/urdf/config/kinect/turtlebot_gazebo.urdf.xacro"/>
+  <xacro:include filename="$(find lab_turtlebot_description)/urdf/config/kinect/turtlebot_properties.urdf.xacro"/>
   <xacro:property name="kinect_cam_py" value="-0.0125"/>
   <!-- Parameterised in part by the values in turtlebot_properties.urdf.xacro -->
-  <xacro:macro name="sensor_steleo" params="parent">
+  <xacro:macro name="sensor_kinect" params="parent">
     <joint name="camera_rgb_joint" type="fixed">
       <origin xyz="${cam_px} ${kinect_cam_py} ${cam_pz}" rpy="${cam_or} ${cam_op} ${cam_oy}"/>
@@ -21,7 +21,7 @@
       <origin xyz="-0.031 ${-kinect_cam_py} -0.016" rpy="0 0 0"/>
       <parent link="camera_rgb_frame"/>
-      <child link="left_camera_frame"/>
+      <child link="camera_link"/>
     </joint>
-      <link name="left_camera_frame">
+      <link name="camera_link">
       <visual>
        <origin xyz="0 0 0" rpy="0 0 ${M_PI/2}"/>

File: lab_turtlebot_description/urdf/config/steleo/steleo.urdf.xacro (robot description, xacro)
@@ -1,9 +1,9 @@
 <?xml version="1.0"?>
-<robot name="sensor_kinect" xmlns:xacro="http://ros.org/wiki/xacro">
-  <xacro:include filename="$(find turtlebot_description)/urdf/turtlebot_gazebo.urdf.xacro"/>
-  <xacro:include filename="$(find lab_turtlebot_description)/urdf/urg/config/turtlebot_properties.urdf.xacro"/>
+<robot name="sensor_steleo" xmlns:xacro="http://ros.org/wiki/xacro">
+  <xacro:include filename="$(find lab_turtlebot_description)/urdf/config/steleo/turtlebot_gazebo.urdf.xacro"/>
+  <xacro:include filename="$(find lab_turtlebot_description)/urdf/config/steleo/turtlebot_properties.urdf.xacro"/>
   <xacro:property name="kinect_cam_py" value="-0.0125"/>
   <!-- Parameterised in part by the values in turtlebot_properties.urdf.xacro -->
-  <xacro:macro name="sensor_kinect" params="parent">
+  <xacro:macro name="sensor_steleo" params="parent">
     <joint name="camera_rgb_joint" type="fixed">
       <origin xyz="${cam_px} ${kinect_cam_py} ${cam_pz}" rpy="${cam_or} ${cam_op} ${cam_oy}"/>
@@ -21,7 +21,7 @@
       <origin xyz="-0.031 ${-kinect_cam_py} -0.016" rpy="0 0 0"/>
       <parent link="camera_rgb_frame"/>
-      <child link="camera_link"/>
+      <child link="left_camera_frame"/>
     </joint>
-      <link name="camera_link">
+      <link name="left_camera_frame">
       <visual>
        <origin xyz="0 0 0" rpy="0 0 ${M_PI/2}"/>

File: lab_turtlebot_description/urdf/config/steleo/turtlebot_common_library.urdf.xacro (robot description, xacro)
@@ -6,4 +6,4 @@
   <!-- General -->
   <xacro:include filename="$(find lab_turtlebot_description)/urdf/config/common_properties.urdf.xacro"/>
-  <xacro:include filename="$(find lab_turtlebot_description)/urdf/config/turtlebot_properties.urdf.xacro"/>
+  <xacro:include filename="$(find lab_turtlebot_description)/urdf/config/steleo/turtlebot_properties.urdf.xacro"/>
 </robot>

File: lab_turtlebot_description/urdf/config/steleo/turtlebot_gazebo.urdf.xacro (robot description, xacro)
@@ -44,5 +44,5 @@
         <alwaysOn>true</alwaysOn>
         <updateRate>0.0</updateRate>
-        <cameraName>multisense_sl/camera</cameraName>
+        <cameraName>camera</cameraName>
         <imageTopicName>image_raw</imageTopicName>
         <cameraInfoTopicName>camera_info</cameraInfoTopicName>

File: lab_turtlebot_description/urdf/config/urg_plus_kinect/kinect.urdf.xacro (robot description, xacro)
@@ -1,6 +1,6 @@
 <?xml version="1.0"?>
 <robot name="sensor_kinect" xmlns:xacro="http://ros.org/wiki/xacro">
-  <xacro:include filename="$(find lab_turtlebot_description)/urdf/config/turtlebot_gazebo_kinect.urdf.xacro"/>
-  <xacro:include filename="$(find lab_turtlebot_description)/urdf/config/turtlebot_properties.urdf.xacro"/>
+  <xacro:include filename="$(find lab_turtlebot_description)/urdf/config/kinect/turtlebot_gazebo.urdf.xacro"/>
+  <xacro:include filename="$(find lab_turtlebot_description)/urdf/config/urg_plus_kinect/turtlebot_properties.urdf.xacro"/>
   <xacro:property name="kinect_cam_py" value="-0.0125"/>
   <!-- Parameterised in part by the values in turtlebot_properties.urdf.xacro -->

File: lab_turtlebot_description/urdf/config/urg_plus_kinect/turtlebot_common_library.urdf.xacro (robot description, xacro)
@@ -6,4 +6,4 @@
   <!-- General -->
   <xacro:include filename="$(find turtlebot_description)/urdf/common_properties.urdf.xacro"/>
-  <xacro:include filename="$(find lab_turtlebot_description)/urdf/config/urg/turtlebot_properties.urdf.xacro"/>
+  <xacro:include filename="$(find lab_turtlebot_description)/urdf/config/urg_plus_kinect/turtlebot_properties.urdf.xacro"/>
 </robot>

File: lab_turtlebot_description/urdf/config/urg_plus_kinect/urg.urdf.xacro (robot description, xacro)
@@ -1,5 +1,5 @@
 <?xml version="1.0"?>
 <robot name="sensor_urg" xmlns:xacro="http://ros.org/wiki/xacro">
-  <xacro:include filename="$(find lab_turtlebot_description)/urdf/config/urg/turtlebot_properties.urdf.xacro"/>
+  <xacro:include filename="$(find lab_turtlebot_description)/urdf/config/urg_plus_kinect/turtlebot_properties.urdf.xacro"/>
   <xacro:macro name="sensor_urg" params="parent">
     <joint name="urg_joint" type="fixed">

File: lab_turtlebot_description/urdf/lab_turtlebot_kinect.urdf.xacro (robot description, xacro)
@@ -6,8 +6,8 @@
 -->
 <robot name="turtlebot" xmlns:xacro="http://ros.org/wiki/xacro">
-  <xacro:include filename="$(find lab_turtlebot_description)/urdf/config/turtlebot_common_library.urdf.xacro" />
+  <xacro:include filename="$(find lab_turtlebot_description)/urdf/config/kinect/turtlebot_common_library.urdf.xacro" />
   <xacro:include filename="$(find lab_turtlebot_description)/urdf/config/kobuki.urdf.xacro" />
   <xacro:include filename="$(find lab_turtlebot_description)/urdf/config/hexagons.urdf.xacro"/>
-  <xacro:include filename="$(find lab_turtlebot_description)/urdf/config/kinect.urdf.xacro"/>
+  <xacro:include filename="$(find lab_turtlebot_description)/urdf/config/kinect/kinect.urdf.xacro"/>
   <kobuki/>
   <stack_hexagons parent="base_link"/>

File: lab_turtlebot_description/urdf/lab_turtlebot_steleo.urdf.xacro (robot description, xacro)
@@ -6,8 +6,8 @@
 -->
 <robot name="turtlebot" xmlns:xacro="http://ros.org/wiki/xacro">
-  <xacro:include filename="$(find lab_turtlebot_description)/urdf/config/turtlebot_common_library.urdf.xacro" />
+  <xacro:include filename="$(find lab_turtlebot_description)/urdf/config/steleo/turtlebot_common_library.urdf.xacro" />
   <xacro:include filename="$(find lab_turtlebot_description)/urdf/config/kobuki.urdf.xacro" />
   <xacro:include filename="$(find lab_turtlebot_description)/urdf/config/hexagons.urdf.xacro"/>
-  <xacro:include filename="$(find lab_turtlebot_description)/urdf/config/steleo.urdf.xacro"/>
+  <xacro:include filename="$(find lab_turtlebot_description)/urdf/config/steleo/steleo.urdf.xacro"/>
   <kobuki/>
   <stack_hexagons parent="base_link"/>
