Commit message: add gazebo steleo

File: lab_turtlebot_description/urdf/config/kinect/turtlebot_properties.urdf.xacro (robot description, xacro)
@@ -19,5 +19,5 @@
      (currently in development and awaiting feedback)
    -->
-   <xacro:include filename="$(find turtlebot_description)/urdf/common_properties.urdf.xacro"/>
+   <xacro:include filename="$(find lab_turtlebot_description)/urdf/config/common_properties.urdf.xacro"/>
   <xacro:property name="cam_px" value="-0.035" />
   <!-- <xacro:property name="cam_px" value="0" /> -->

File: lab_turtlebot_description/urdf/config/steleo/steleo.urdf.xacro (robot description, xacro)
@@ -3,62 +3,52 @@
   <xacro:include filename="$(find lab_turtlebot_description)/urdf/config/steleo/turtlebot_gazebo.urdf.xacro"/>
   <xacro:include filename="$(find lab_turtlebot_description)/urdf/config/steleo/turtlebot_properties.urdf.xacro"/>
-  <xacro:property name="kinect_cam_py" value="-0.0125"/>
-  <!-- Parameterised in part by the values in turtlebot_properties.urdf.xacro -->
+  <xacro:property name="steleo_cam_py" value="-0.0125"/>
   <xacro:macro name="sensor_steleo" params="parent">
-    <joint name="camera_rgb_joint" type="fixed">
-      <origin xyz="${cam_px} ${kinect_cam_py} ${cam_pz}" rpy="${cam_or} ${cam_op} ${cam_oy}"/>
-      <parent link="${parent}"/>
-      <child link="camera_rgb_frame" />
+    <!-- Camera Center -->
+    <joint name="camera_center_joint" type="fixed">
+        <parent link="${parent}"/>
+        <child link="camera_center_frame"/>
+        <origin xyz="${cam_px} ${steleo_cam_py} ${cam_pz}" rpy="${cam_or} ${cam_op} ${cam_oy}"/>
     </joint>
-    <link name="camera_rgb_frame"/>
-    <joint name="camera_rgb_optical_joint" type="fixed">
-      <origin xyz="0 0 0" rpy="${-M_PI/2} 0 ${-M_PI/2}" />
-      <parent link="camera_rgb_frame" />
-      <child link="camera_rgb_optical_frame" />
+    <link name="camera_center_frame">
+        <visual>
+            <origin xyz="0 0 0" rpy="0 0 0"/>
+            <geometry>
+                <mesh filename="package://lab_turtlebot_description/urdf/config/steleo/steleo.stl" />
+            </geometry>
+            <material name="light_grey">
+                <color rgba="0.8 0.8 0.8 0.8"/>
+            </material>
+        </visual>
+    </link>
+  <!-- Left Camera -->
+    <joint name="left_camera_joint" type="fixed">
+        <parent link="camera_center_frame"/>
+        <child link="left_camera_frame"/>
+        <origin xyz="0 0.06 0" rpy="0 0 0" />
     </joint>
-    <link name="camera_rgb_optical_frame"/>
-    <joint name="camera_joint" type="fixed">
-      <origin xyz="-0.031 ${-kinect_cam_py} -0.016" rpy="0 0 0"/>
-      <parent link="camera_rgb_frame"/>
-      <child link="left_camera_frame"/>
+    <link name="left_camera_frame" />
+    <joint name="left_camera_optical_joint" type="fixed">
+        <origin xyz="0 0 0" rpy="-1.57079632679 0.0 -1.57079632679"/>
+        <parent link="left_camera_frame"/>
+        <child link="left_camera_optical_frame"/>
     </joint>
-      <link name="left_camera_frame">
-      <visual>
-       <origin xyz="0 0 0" rpy="0 0 ${M_PI/2}"/>
-        <geometry>
-         <mesh filename="package://turtlebot_description/meshes/sensors/kinect.dae"/>
-        </geometry>
-      </visual>
-  	  <collision>
-        <origin xyz="0.0 0.0 0.0" rpy="0 0 0"/>
-  	    <geometry>
-  	      <box size="0.07271 0.27794 0.073"/>
-  	    </geometry>
-  	  </collision>
-      <inertial>
-        <mass value="0.564" />
-        <origin xyz="0 0 0" />
-        <inertia ixx="0.003881243" ixy="0.0" ixz="0.0"
-                 iyy="0.000498940" iyz="0.0"
-                 izz="0.003879257" />
-      </inertial>
-    </link>
-    <!-- The fixed joints & links below are usually published by static_transformers launched by the OpenNi launch
-         files. However, for Gazebo simulation we need them, so we add them here.
-         (Hence, don't publish them additionally!) -->
-	<joint name="camera_depth_joint" type="fixed">
-	  <origin xyz="0 ${2 * -kinect_cam_py} 0" rpy="0 0 0" />
-	  <parent link="camera_rgb_frame" />
-	  <child link="camera_depth_frame" />
-	</joint>
-	<link name="camera_depth_frame"/>
-	<joint name="camera_depth_optical_joint" type="fixed">
-	  <origin xyz="0 0 0" rpy="${-M_PI/2} 0 ${-M_PI/2}" />
-	  <parent link="camera_depth_frame" />
-	  <child link="camera_depth_optical_frame" />
-	</joint>
-	<link name="camera_depth_optical_frame"/>
-	<!-- Kinect sensor for simulation -->
-	<turtlebot_sim_3dsensor/>
+    <link name="left_camera_optical_frame"/>
+  <!-- Right Camera -->
+    <joint name="right_camera_joint" type="fixed">
+        <parent link="camera_center_frame"/>
+        <child link="right_camera_frame"/>
+        <origin xyz="0 -0.06 0" rpy="0 0 0" />
+    </joint>
+    <link name="right_camera_frame" />
+    <joint name="right_camera_optical_joint" type="fixed">
+        <origin xyz="0 0 0" rpy="-1.57079632679 0.0 -1.57079632679"/>
+        <parent link="right_camera_frame"/>
+        <child link="right_camera_optical_frame"/>
+    </joint>
+    <link name="right_camera_optical_frame"/>
+	<!-- steleo sensor for simulation -->
+    <turtlebot_sim_steleo_left/>
+    <turtlebot_sim_steleo_right/>
   </xacro:macro>
 </robot>

File: lab_turtlebot_description/urdf/config/steleo/turtlebot_gazebo.urdf.xacro (robot description, xacro)
@@ -1,53 +1,79 @@
 <?xml version="1.0"?>
+<!-- detail of parameters : http://docs.ros.org/kinetic/api/gazebo_plugins/html/gazebo__ros__camera__utils_8cpp_source.html-->
 <robot name="turtlebot_gazebo" xmlns:xacro="http://ros.org/wiki/xacro">
-  <!-- Microsoft Kinect / ASUS Xtion PRO Live for simulation -->
-  <xacro:macro name="turtlebot_sim_3dsensor">
+  <xacro:property name="WIDTH" value="1280" />
+  <xacro:property name="HEIGHT" value="720" />
+  <xacro:property name="UPDATE_RATE" value="30.0" />
+  <xacro:property name="HORIZONTAL_FOV" value="1.3962634" />
+  <xacro:property name="CLIP_NEAR" value="0.02" />
+  <xacro:property name="CLIP_FAR" value="300" />
+  <xacro:property name="HACK_BASE_LINE" value="0.07" />
+  <xacro:macro name="turtlebot_sim_steleo_left">
     <gazebo reference="left_camera_frame">
-    <sensor type="multicamera" name="stereo_camera">
-      <update_rate>30.0</update_rate>
+    <sensor type="camera" name="stereo_camera_left">
+      <update_rate>${UPDATE_RATE}</update_rate>
       <camera name="left">
-        <horizontal_fov>1.3962634</horizontal_fov>
+        <horizontal_fov>${HORIZONTAL_FOV}</horizontal_fov>
         <image>
-          <width>800</width>
-          <height>800</height>
+          <width>${WIDTH}</width>
+          <height>${HEIGHT}</height>
           <format>R8G8B8</format>
         </image>
         <clip>
-          <near>0.02</near>
-          <far>300</far>
+          <near>${CLIP_NEAR}</near>
+          <far>${CLIP_FAR}</far>
         </clip>
-        <noise>
+        <!-- <noise>
           <type>gaussian</type>
           <mean>0.0</mean>
           <stddev>0.007</stddev>
-        </noise>
+        </noise> -->
       </camera>
+      <plugin name="stereo_camera_left_controller" filename="libgazebo_ros_camera.so">
+        <alwaysOn>true</alwaysOn>
+        <updateRate>0.0</updateRate>
+        <cameraName>camera/left</cameraName>
+        <imageTopicName>image_raw</imageTopicName>
+        <cameraInfoTopicName>camera_info</cameraInfoTopicName>
+        <frameName>left_camera_optical_frame</frameName>
+        <hackBaseline>${HACK_BASE_LINE}</hackBaseline>
+        <distortionK1>0.0</distortionK1>
+        <distortionK2>0.0</distortionK2>
+        <distortionK3>0.0</distortionK3>
+        <distortionT1>0.0</distortionT1>
+        <distortionT2>0.0</distortionT2>
+      </plugin>
+    </sensor>
+  </gazebo>
+  </xacro:macro>
+  <xacro:macro name="turtlebot_sim_steleo_right">
+    <gazebo reference="right_camera_frame">
+    <sensor type="camera" name="stereo_camera_right">
+      <update_rate>${UPDATE_RATE}</update_rate>
       <camera name="right">
-        <pose>0 -0.07 0 0 0 0</pose>
-        <horizontal_fov>1.3962634</horizontal_fov>
+        <horizontal_fov>${HORIZONTAL_FOV}</horizontal_fov>
         <image>
-          <width>800</width>
-          <height>800</height>
+          <width>${WIDTH}</width>
+          <height>${HEIGHT}</height>
           <format>R8G8B8</format>
         </image>
         <clip>
-          <near>0.02</near>
-          <far>300</far>
+          <near>${CLIP_NEAR}</near>
+          <far>${CLIP_FAR}</far>
         </clip>
-        <noise>
+        <!-- <noise>
           <type>gaussian</type>
           <mean>0.0</mean>
           <stddev>0.007</stddev>
-        </noise>
+        </noise> -->
       </camera>
-      <plugin name="stereo_camera_controller" filename="libgazebo_ros_multicamera.so">
+      <plugin name="stereo_camera_right_controller" filename="libgazebo_ros_camera.so">
         <alwaysOn>true</alwaysOn>
         <updateRate>0.0</updateRate>
-        <cameraName>camera</cameraName>
+        <cameraName>camera/right</cameraName>
         <imageTopicName>image_raw</imageTopicName>
         <cameraInfoTopicName>camera_info</cameraInfoTopicName>
-        <frameName>left_camera_optical_frame</frameName>
-        <!--<rightFrameName>right_camera_optical_frame</rightFrameName>-->
-        <hackBaseline>0.07</hackBaseline>
+        <frameName>right_camera_optical_frame</frameName>
+        <hackBaseline>${HACK_BASE_LINE}</hackBaseline>
         <distortionK1>0.0</distortionK1>
         <distortionK2>0.0</distortionK2>

File: lab_turtlebot_description/urdf/config/urg_plus_kinect/turtlebot_properties.urdf.xacro (robot description, xacro)
@@ -19,5 +19,5 @@
      (currently in development and awaiting feedback)
    -->
-   <xacro:include filename="$(find turtlebot_description)/urdf/common_properties.urdf.xacro"/>
+   <xacro:include filename="$(find lab_turtlebot_description)/urdf/config/common_properties.urdf.xacro"/>
   <!-- <xacro:property name="cam_px" value="-0.035" /> -->
   <xacro:property name="cam_px" value="0.07" />
