Commit message: minor fix

File: lab_turtlebot_description/urdf/config/steleo/steleo.urdf.xacro (robot description, xacro)
@@ -3,5 +3,4 @@
   <xacro:include filename="$(find lab_turtlebot_description)/urdf/config/steleo/turtlebot_gazebo.urdf.xacro"/>
   <xacro:include filename="$(find lab_turtlebot_description)/urdf/config/steleo/turtlebot_properties.urdf.xacro"/>
-  <xacro:property name="steleo_cam_py" value="-0.0125"/>
   <xacro:macro name="sensor_steleo" params="parent">
     <!-- Camera Center -->
@@ -9,5 +8,5 @@
         <parent link="${parent}"/>
         <child link="camera_center_frame"/>
-        <origin xyz="${cam_px} ${steleo_cam_py} ${cam_pz}" rpy="${cam_or} ${cam_op} ${cam_oy}"/>
+        <origin xyz="${cam_px} ${cam_py} ${cam_pz}" rpy="${cam_or} ${cam_op} ${cam_oy}"/>
     </joint>
     <link name="camera_center_frame">

File: lab_turtlebot_description/urdf/config/steleo/turtlebot_properties.urdf.xacro (robot description, xacro)
@@ -21,9 +21,6 @@
    <xacro:include filename="$(find lab_turtlebot_description)/urdf/config/common_properties.urdf.xacro"/>
   <xacro:property name="cam_px" value="-0.035" />
-  <!-- <xacro:property name="cam_px" value="0" /> -->
-  <!-- <xacro:property name="cam_px" value="0.00" /> -->
-<!--	<xacro:property name="cam_py" value="-0.0125" /> Y varies for different configurations. get sets in sensors_urdf -->
+	<xacro:property name="cam_py" value="-0.0125" />
   <xacro:property name="cam_pz" value="0.390" />
-  <!-- <xacro:property name="cam_pz" value="0" /> -->
 	<xacro:property name="cam_or" value="0" />
 	<xacro:property name="cam_op" value="0" />
