Commit message: update urdf and gazebo launch

File: lab_turtlebot_description/urdf/config/urg_plus_kinect/kinect.urdf.xacro (robot description, xacro)
@@ -1,5 +1,5 @@
 <?xml version="1.0"?>
 <robot name="sensor_kinect" xmlns:xacro="http://ros.org/wiki/xacro">
-  <xacro:include filename="$(find lab_turtlebot_description)/urdf/config/kinect/turtlebot_gazebo.urdf.xacro"/>
+  <xacro:include filename="$(find lab_turtlebot_description)/urdf/config/urg_plus_kinect/turtlebot_gazebo.urdf.xacro"/>
   <xacro:include filename="$(find lab_turtlebot_description)/urdf/config/urg_plus_kinect/turtlebot_properties.urdf.xacro"/>
   <xacro:property name="kinect_cam_py" value="-0.0125"/>

File: lab_turtlebot_description/urdf/config/urg_plus_kinect/kobuki.urdf.xacro (robot description, xacro)
@@ -61,6 +61,5 @@
       <origin xyz="-0.10 0 0.38" rpy="0 0 0"/>
     </joint>
-    <link name="merge_laser_link">
-    </link>
+    <link name="merge_laser_link"/>
     <joint name="wheel_left_joint" type="continuous">
       <parent link="base_link"/>

File: lab_turtlebot_description/urdf/config/urg_plus_kinect/urg.urdf.xacro (robot description, xacro)
@@ -1,4 +1,5 @@
 <?xml version="1.0"?>
 <robot name="sensor_urg" xmlns:xacro="http://ros.org/wiki/xacro">
+  <xacro:include filename="$(find lab_turtlebot_description)/urdf/config/urg_plus_kinect/turtlebot_gazebo.urdf.xacro"/>
   <xacro:include filename="$(find lab_turtlebot_description)/urdf/config/urg_plus_kinect/turtlebot_properties.urdf.xacro"/>
   <xacro:macro name="sensor_urg" params="parent">
@@ -8,5 +9,13 @@
       <child link="urg_frame" />
     </joint>
-    <link name="urg_frame"/>
+    <link name="urg_frame">
+      <visual>
+          <origin xyz="0 0 0" rpy="0 0 0"/>
+          <geometry>
+              <mesh filename="package://lab_turtlebot_description/urdf/config/steleo/steleo.stl" />
+          </geometry>
+      </visual>
+    </link>
+    <turtlebot_sim_urg/>
   </xacro:macro>
 </robot>
