Commit message: laser test

File: lab_turtlebot_description/urdf/config/urg_plus_kinect/turtlebot_gazebo.urdf.xacro (robot description, xacro)
@@ -57,5 +57,5 @@
           <range>
             <min>0.05</min>
-            <max>30.0</max>
+            <max>50.0</max>
             <resolution>0.01</resolution>
           </range>

File: lab_turtlebot_description/urdf/config/urg_plus_kinect/turtlebot_properties.urdf.xacro (robot description, xacro)
@@ -29,9 +29,11 @@
 	<xacro:property name="cam_op" value="0" />
 	<xacro:property name="cam_oy" value="0" />
-  <xacro:property name="urg_px" value="-0.06" />
+  <!-- <xacro:property name="urg_px" value="-0.06" /> -->
+  <xacro:property name="urg_px" value="0.1" />
 	<xacro:property name="urg_py" value="0.0" />
-  <xacro:property name="urg_pz" value="0.0" />
+  <xacro:property name="urg_pz" value="0.15" />
 	<xacro:property name="urg_or" value="0.0" />
 	<xacro:property name="urg_op" value="0.0" />
-	<xacro:property name="urg_oy" value="${M_PI}" />
+	<!-- <xacro:property name="urg_oy" value="${M_PI}" /> -->
+  <xacro:property name="urg_oy" value="0.0" />
 </robot>
