Commit message: typo

File: lab_turtlebot_description/urdf/config/stereo/stereo.urdf.xacro (robot description, xacro)
@@ -1,7 +1,7 @@
 <?xml version="1.0"?>
-<robot name="sensor_steleo" xmlns:xacro="http://ros.org/wiki/xacro">
-  <xacro:include filename="$(find lab_turtlebot_description)/urdf/config/steleo/turtlebot_gazebo.urdf.xacro"/>
-  <xacro:include filename="$(find lab_turtlebot_description)/urdf/config/steleo/turtlebot_properties.urdf.xacro"/>
-  <xacro:macro name="sensor_steleo" params="parent">
+<robot name="sensor_stereo" xmlns:xacro="http://ros.org/wiki/xacro">
+  <xacro:include filename="$(find lab_turtlebot_description)/urdf/config/stereo/turtlebot_gazebo.urdf.xacro"/>
+  <xacro:include filename="$(find lab_turtlebot_description)/urdf/config/stereo/turtlebot_properties.urdf.xacro"/>
+  <xacro:macro name="sensor_stereo" params="parent">
     <!-- Camera Center -->
     <joint name="camera_center_joint" type="fixed">
@@ -14,5 +14,5 @@
             <origin xyz="0 0 0" rpy="0 0 0"/>
             <geometry>
-                <mesh filename="package://lab_turtlebot_description/urdf/config/steleo/steleo.stl" />
+                <mesh filename="package://lab_turtlebot_description/urdf/config/stereo/stereo.stl" />
             </geometry>
             <material name="light_grey">
@@ -47,7 +47,7 @@
     </joint>
     <link name="right_camera_optical_frame"/>
-	<!-- steleo sensor for simulation -->
-    <turtlebot_sim_steleo_left/>
-    <turtlebot_sim_steleo_right/>
+	<!-- stereo sensor for simulation -->
+    <turtlebot_sim_stereo_left/>
+    <turtlebot_sim_stereo_right/>
   </xacro:macro>
 </robot>

File: lab_turtlebot_description/urdf/config/stereo/turtlebot_common_library.urdf.xacro (robot description, xacro)
@@ -6,4 +6,4 @@
   <!-- General -->
   <xacro:include filename="$(find lab_turtlebot_description)/urdf/config/common_properties.urdf.xacro"/>
-  <xacro:include filename="$(find lab_turtlebot_description)/urdf/config/steleo/turtlebot_properties.urdf.xacro"/>
+  <xacro:include filename="$(find lab_turtlebot_description)/urdf/config/stereo/turtlebot_properties.urdf.xacro"/>
 </robot>

File: lab_turtlebot_description/urdf/config/stereo/turtlebot_gazebo.urdf.xacro (robot description, xacro)
@@ -9,5 +9,5 @@
   <xacro:property name="CLIP_FAR" value="300" />
   <xacro:property name="HACK_BASE_LINE" value="0.07" />
-  <xacro:macro name="turtlebot_sim_steleo_left">
+  <xacro:macro name="turtlebot_sim_stereo_left">
     <gazebo reference="left_camera_frame">
     <sensor type="camera" name="stereo_camera_left">
@@ -47,5 +47,5 @@
   </gazebo>
   </xacro:macro>
-  <xacro:macro name="turtlebot_sim_steleo_right">
+  <xacro:macro name="turtlebot_sim_stereo_right">
     <gazebo reference="right_camera_frame">
     <sensor type="camera" name="stereo_camera_right">

File: lab_turtlebot_description/urdf/config/urg_plus_kinect/turtlebot_gazebo.urdf.xacro (robot description, xacro)
@@ -43,5 +43,5 @@
   <xacro:macro name="turtlebot_sim_urg">
     <gazebo reference="urg_frame">
-      <sesnor type="ray" name="urg">
+      <sensor type="ray" name="urg">
         <always_on>true</always_on>
         <update_rate>30.0</update_rate>
@@ -62,5 +62,5 @@
         </ray>
         <plugin name="urg_controller" filename="libgazebo_ros_laser.so">
-          <topicName>scan</topicName>
+          <topicName>urg_scan</topicName>
           <frameName>urg_frame</frameName>
         </plugin>

File: lab_turtlebot_description/urdf/config/urg_plus_kinect/urg.urdf.xacro (robot description, xacro)
@@ -13,5 +13,5 @@
           <origin xyz="0 0 0" rpy="0 0 0"/>
           <geometry>
-              <mesh filename="package://lab_turtlebot_description/urdf/config/steleo/steleo.stl" />
+              <mesh filename="package://lab_turtlebot_description/urdf/config/stereo/stereo.stl" />
           </geometry>
       </visual>

File: lab_turtlebot_description/urdf/lab_turtlebot_stereo.urdf.xacro (robot description, xacro)
@@ -6,10 +6,10 @@
 -->
 <robot name="turtlebot" xmlns:xacro="http://ros.org/wiki/xacro">
-  <xacro:include filename="$(find lab_turtlebot_description)/urdf/config/steleo/turtlebot_common_library.urdf.xacro" />
+  <xacro:include filename="$(find lab_turtlebot_description)/urdf/config/stereo/turtlebot_common_library.urdf.xacro" />
   <xacro:include filename="$(find lab_turtlebot_description)/urdf/config/kobuki.urdf.xacro" />
   <xacro:include filename="$(find lab_turtlebot_description)/urdf/config/hexagons.urdf.xacro"/>
-  <xacro:include filename="$(find lab_turtlebot_description)/urdf/config/steleo/steleo.urdf.xacro"/>
+  <xacro:include filename="$(find lab_turtlebot_description)/urdf/config/stereo/stereo.urdf.xacro"/>
   <kobuki/>
   <stack_hexagons parent="base_link"/>
-  <sensor_steleo  parent="base_link"/>
+  <sensor_stereo  parent="base_link"/>
 </robot>
